Commit message: description: introducing virtual walls around table
Signed-off-by: Wolfgang Wiedmeyer <wolfgang.wiedmeyer@kit.edu>

File: rll_description/urdf/iiwa_table.urdf.xacro (robot description, xacro)
@@ -10,4 +10,7 @@
   <material name="steel">
     <color rgba="0.8784 0.8745 0.8588 1.0"/>
+  </material>
+  <material name="transparent">
+    <color rgba="0.8784 0.8745 0.8588 0.3"/>
   </material>
   <!--  Define the origin of your 3D space
@@ -31,5 +34,103 @@
     </collision>
   </link>
+  <!-- virtual walls
+  Every wall is a link which does not collude with a different wall or the collision link of the steel plate -->
+  <joint name="wall_joint1" type="fixed">
+    <parent link="world" />
+    <child link="wall_front" />
+    <origin xyz="0.605 0 0.7" rpy="0 0 0"/>
+  </joint>
+  <joint name="wall_joint2" type="fixed">
+    <parent link="world" />
+    <child link="wall_back" />
+    <origin xyz="-0.605 0 0.7" rpy="0 0 0"/>
+  </joint>
+  <joint name="wall_joint3" type="fixed">
+    <parent link="world" />
+    <child link="wall_left" />
+    <origin xyz="0 -0.805 0.7" rpy="0 0 0"/>
+  </joint>
+  <joint name="wall_joint4" type="fixed">
+    <parent link="world" />
+    <child link="wall_right" />
+    <origin xyz="0 0.805 0.7" rpy="0 0 0"/>
+  </joint>
+  <link name="wall_front">
+    <visual>
+      <origin xyz="0 0 0" rpy="0 0 0"/>
+      <geometry>
+        <box size="0.01 1.599 1.1" rpy="0 0 0"/>
+      </geometry>
+      <material name="transparent" />
+    </visual>
+    <collision>
+      <origin xyz="0 0 0" rpy="0 0 0"/>
+      <geometry>
+        <box size="0.01 1.599 1.1" rpy="0 0 0"/>
+      </geometry>
+      <material name="transparent" />
+    </collision>
+  </link>
+  <link name="wall_back">
+    <visual>
+      <origin xyz="0 0 0" rpy="0 0 0"/>
+      <geometry>
+        <box size="0.01 1.599 1.1" rpy="0 0 0"/>
+      </geometry>
+      <material name="transparent" />
+    </visual>
+    <collision>
+      <origin xyz="0 0 0" rpy="0 0 0"/>
+      <geometry>
+        <box size="0.01 1.599 1.1" rpy="0 0 0"/>
+      </geometry>
+      <material name="transparent" />
+    </collision>
+  </link>
+  <link name="wall_left">
+    <visual>
+      <origin xyz="0 0 0" rpy="0 0 0"/>
+      <geometry>
+        <box size="1.199 0.01 1.1" rpy="0 0 0"/>
+      </geometry>
+      <material name="transparent" />
+    </visual>
+    <collision>
+      <origin xyz="0 0 0" rpy="0 0 0"/>
+      <geometry>
+        <box size="1.199 0.01 1.1" rpy="0 0 0"/>
+      </geometry>
+      <material name="transparent" />
+    </collision>
+  </link>
+  <link name="wall_right">
+    <visual>
+      <origin xyz="0 0 0" rpy="0 0 0"/>
+      <geometry>
+        <box size="1.199 0.01 1.1" rpy="0 0 0"/>
+      </geometry>
+      <material name="transparent" />
+    </visual>
+    <collision>
+      <origin xyz="0 0 0" rpy="0 0 0"/>
+      <geometry>
+        <box size="1.199 0.01 1.1" rpy="0 0 0"/>
+      </geometry>
+      <material name="transparent" />
+    </collision>
+  </link>
   <gazebo reference="world">
+    <static>true</static>
+  </gazebo>
+  <gazebo reference="wall_front">
+    <static>true</static>
+  </gazebo>
+  <gazebo reference="wall_back">
+    <static>true</static>
+  </gazebo>
+  <gazebo reference="wall_left">
+    <static>true</static>
+  </gazebo>
+  <gazebo reference="wall_right">
     <static>true</static>
   </gazebo>

Commit message: description and two iiwas moveit: add gripper in a rudimentary fashion
Signed-off-by: Wolfgang Wiedmeyer <wolfgang.wiedmeyer@kit.edu>

File: rll_description/urdf/iiwa_table.urdf.xacro (robot description, xacro)
@@ -5,4 +5,6 @@
   <!--Import the iiwa7 macro -->
   <xacro:include filename="$(find iiwa_description)/urdf/iiwa7.xacro"/>
+  <!--Import the schunk gripper egl90  -->
+  <xacro:include filename="$(find schunk_gripper_egl90)/urdf/egl90_macro.xacro"/>
   <!--  Arguments for the iiwa7 macro  -->
   <xacro:arg name="hardware_interface" default="PositionJointInterface"/>
@@ -139,3 +141,10 @@
     <origin xyz="0 0 0" rpy="0 0 0"/>
   </xacro:iiwa7>
+  <!-- Here we insert a schunk gripper in the scene -->
+   <xacro:egl90 parent="$(arg robot_name)_link_ee" prefix="$(arg robot_name)_">
+      <origin xyz="0 0 0.02" rpy="0 0 0"/>
+   </xacro:egl90>
+   <xacro:egl90-jaws prefix="$(arg robot_name)_" x="0.0" min="-0.015" max="0.026">
+     <mesh filename="package://schunk_gripper_egl90/meshes/finger.stl"/>
+   </xacro:egl90-jaws>
 </robot>

Commit message: add our gripper adapter and fingers
Signed-off-by: Wolfgang Wiedmeyer <wolfgang.wiedmeyer@kit.edu>

File: rll_description/urdf/iiwa_table.urdf.xacro (robot description, xacro)
@@ -17,6 +17,6 @@
   </material>
   <!--  Define the origin of your 3D space
-  Here we define a box lying at 0,0,0 with some dimensions. In reality, our robot is placed on top of a steel table.
-  This will include the table top in the scene and avoid the robot to hit it when using MoveIt!
+       Here we define a box lying at 0,0,0 with some dimensions. In reality, our robot is placed on top of a steel table.
+       This will include the table top in the scene and avoid the robot to hit it when using MoveIt!
   -->
   <link name="world">
@@ -37,5 +37,5 @@
   </link>
   <!-- virtual walls
-  Every wall is a link which does not collide with a different wall or the collision link of the steel plate -->
+       Every wall is a link which does not collide with a different wall or the collision link of the steel plate -->
   <joint name="wall_joint1" type="fixed">
     <parent link="world" />
@@ -142,9 +142,30 @@
   </xacro:iiwa7>
   <!-- Here we insert a schunk gripper in the scene -->
-   <xacro:egl90 parent="$(arg robot_name)_link_ee" prefix="$(arg robot_name)_">
-      <origin xyz="0 0 0.02" rpy="0 0 0"/>
-   </xacro:egl90>
-   <xacro:egl90-jaws prefix="$(arg robot_name)_" x="0.0" min="-0.015" max="0.026">
-     <mesh filename="package://schunk_gripper_egl90/meshes/finger.stl"/>
-   </xacro:egl90-jaws>
+  <joint name="gripper_adapter_joint" type="fixed">
+    <parent link="$(arg robot_name)_link_ee" />
+    <child link="$(arg robot_name)_gripper_adapter" />
+    <origin xyz="0 0 0" rpy="0 0 0"/>
+  </joint>
+  <link name="$(arg robot_name)_gripper_adapter">
+    <visual>
+      <origin xyz="0 0 0.024" rpy="${180 * PI / 180} 0 ${-90 * PI / 180}"/>
+      <geometry>
+        <mesh filename="package://rll_description/meshes/visual/gripper_adapter.dae" scale="0.001 0.001 0.001"/>
+      </geometry>
+      <material name="Grey"/>
+    </visual>
+    <collision>
+      <origin xyz="0 0 0.024" rpy="${180 * PI / 180} 0 ${-90 * PI / 180}"/>
+      <geometry>
+        <mesh filename="package://rll_description/meshes/visual/gripper_adapter.dae" scale="0.001 0.001 0.001"/>
+      </geometry>
+      <material name="Grey"/>
+    </collision>
+  </link>
+  <xacro:egl90 parent="$(arg robot_name)_gripper_adapter" prefix="$(arg robot_name)_">
+    <origin xyz="0 0 0.024" rpy="0 0 ${-90 * PI / 180}"/>
+  </xacro:egl90>
+  <xacro:egl90-jaws prefix="$(arg robot_name)_" x="0.0" min="-0.015" max="0.026">
+    <mesh filename="package://rll_description/meshes/visual/gripper_finger.dae" scale="0.001 0.001 0.001"/>
+  </xacro:egl90-jaws>
 </robot>

Commit message: simple moveit Pick-and-Place interface
Signed-off-by: Wolfgang Wiedmeyer <wolfgang.wiedmeyer@kit.edu>

File: rll_description/urdf/iiwa_table.urdf.xacro (robot description, xacro)
@@ -31,5 +31,6 @@
       <origin xyz="0 0 -0.1" rpy="0 0 0"/>
       <geometry>
-        <box size="1.2 1.6 0.49"/>
+        <!-- <box size="1.2 1.6 0.49"/> -->
+        <box size="1.2 1.6 0.2"/>
       </geometry>
       <material name="steel" />

Commit message: improved gripper config
Signed-off-by: Wolfgang Wiedmeyer <wolfgang.wiedmeyer@kit.edu>

File: rll_description/urdf/iiwa_table.urdf.xacro (robot description, xacro)
@@ -31,6 +31,8 @@
       <origin xyz="0 0 -0.1" rpy="0 0 0"/>
       <geometry>
+        <!-- for disallowing eef positions below joint 1 -->
         <!-- <box size="1.2 1.6 0.49"/> -->
-        <box size="1.2 1.6 0.2"/>
+        <!-- for grasping objects on table -->
+        <box size="1.2 1.6 0.203"/>
       </geometry>
       <material name="steel" />
@@ -170,3 +172,10 @@
     <mesh filename="package://rll_description/meshes/visual/gripper_finger.dae" scale="0.001 0.001 0.001"/>
   </xacro:egl90-jaws>
+  <!-- TCP link -->
+  <joint name="gripper_ee_joint" type="fixed">
+    <parent link="$(arg robot_name)_link_ee" />
+    <child link="$(arg robot_name)_gripper_link_ee" />
+    <origin xyz="0 0 0.248" rpy="0 0 0"/>
+  </joint>
+  <link name="$(arg robot_name)_gripper_link_ee"/>
 </robot>

Commit message: description: add base adapter and Roboception camera
Signed-off-by: Wolfgang Wiedmeyer <wolfgang.wiedmeyer@kit.edu>

File: rll_description/urdf/iiwa_table.urdf.xacro (robot description, xacro)
@@ -3,8 +3,7 @@
   <!-- Import Rviz colors -->
   <xacro:include filename="$(find iiwa_description)/urdf/materials.xacro" />
-  <!--Import the iiwa7 macro -->
   <xacro:include filename="$(find iiwa_description)/urdf/iiwa7.xacro"/>
-  <!--Import the schunk gripper egl90  -->
   <xacro:include filename="$(find schunk_gripper_egl90)/urdf/egl90_macro.xacro"/>
+  <xacro:include filename="$(find rc_visard_description)/urdf/rc_visard_160.xacro"/>
   <!--  Arguments for the iiwa7 macro  -->
   <xacro:arg name="hardware_interface" default="PositionJointInterface"/>
@@ -140,7 +139,27 @@
     <static>true</static>
   </gazebo>
-  <!-- Here we insert an iiwa7 robot in the scene, it's origin is just on top of the box previously defined. -->
-  <xacro:iiwa7 hardware_interface="$(arg hardware_interface)" robot_name="$(arg robot_name)" parent="world">
-    <origin xyz="0 0 0" rpy="0 0 0"/>
+  <joint name="base_adapter_joint" type="fixed">
+    <parent link="world" />
+    <child link="$(arg robot_name)_base_adapter" />
+    <origin xyz="-0.2 0 0" rpy="0 0 0"/>
+  </joint>
+  <link name="$(arg robot_name)_base_adapter">
+    <visual>
+      <origin xyz="0 0 0.01" rpy="0 0 0"/>
+      <geometry>
+        <cylinder length="0.02" radius="0.16"/>
+      </geometry>
+      <material name="steel" />
+    </visual>
+    <collision>
+      <origin xyz="0 0 0.01" rpy="0 0 0"/>
+      <geometry>
+        <cylinder length="0.02" radius="0.16"/>
+      </geometry>
+    </collision>
+  </link>
+  <!-- Here we insert an iiwa7 robot in the scene, it's origin is on top of the adapter. -->
+  <xacro:iiwa7 hardware_interface="$(arg hardware_interface)" robot_name="$(arg robot_name)" parent="$(arg robot_name)_base_adapter">
+    <origin xyz="0 0 0.02" rpy="0 0 0"/>
   </xacro:iiwa7>
   <!-- Here we insert a schunk gripper in the scene -->
@@ -179,3 +198,26 @@
   </joint>
   <link name="$(arg robot_name)_gripper_link_ee"/>
+  <joint name="roboception_base_joint" type="fixed">
+    <parent link="world" />
+    <child link="roboception_base" />
+    <origin xyz="0.52 0.72 0.74" rpy="0 0 ${135 * PI / 180}"/>
+  </joint>
+  <link name="roboception_base">
+    <visual>
+      <origin xyz="0 0 0.04" rpy="0 0 0"/>
+      <geometry>
+        <cylinder length="0.08" radius="0.03"/>
+      </geometry>
+      <material name="steel" />
+    </visual>
+    <collision>
+      <origin xyz="0 0 0.04" rpy="0 0 0"/>
+      <geometry>
+        <cylinder length="0.08" radius="0.03"/>
+      </geometry>
+    </collision>
+  </link>
+  <xacro:rc_160 parent="roboception_base" prefix="$(arg robot_name)_">
+    <origin xyz="-0.08 0.03 0.1" rpy="${-135 * PI / 180} 0 0"/>
+  </xacro:rc_160>
 </robot>

Commit message: add a collision box for the camera
Signed-off-by: Wolfgang Wiedmeyer <wolfgang.wiedmeyer@kit.edu>

File: rll_description/urdf/iiwa_table.urdf.xacro (robot description, xacro)
@@ -221,3 +221,17 @@
     <origin xyz="-0.08 0.03 0.1" rpy="${-135 * PI / 180} 0 0"/>
   </xacro:rc_160>
+  <joint name="roboception_collision_joint" type="fixed">
+    <parent link="world" />
+    <child link="roboception_collision" />
+    <origin xyz="0.52 0.72 0.74" rpy="0 0 ${135 * PI / 180}"/>
+  </joint>
+  <link name="roboception_collision">
+    <collision>
+      <origin xyz="-0.0 0.03 0.1" rpy="${-135 * PI / 180} 0 0"/>
+      <geometry>
+        <box size="0.30 0.13 0.10" rpy="0 0 0"/>
+      </geometry>
+      <material name="transparent" />
+    </collision>
+  </link>
 </robot>

Commit message: description: smaller visuals for virtual walls
Signed-off-by: Wolfgang Wiedmeyer <wolfgang.wiedmeyer@kit.edu>

File: rll_description/urdf/iiwa_table.urdf.xacro (robot description, xacro)
@@ -16,5 +16,5 @@
   </material>
   <!--  Define the origin of your 3D space
-       Here we define a box lying at 0,0,0 with some dimensions. In reality, our robot is placed on top of a steel table.
+       Here we define a box lying at 0,0,0 with some dimensions. In reality, our robot is placed on top of a table.
        This will include the table top in the scene and avoid the robot to hit it when using MoveIt!
   -->
@@ -38,6 +38,5 @@
     </collision>
   </link>
-  <!-- virtual walls
-       Every wall is a link which does not collide with a different wall or the collision link of the steel plate -->
+  <!-- virtual walls -->
   <joint name="wall_joint1" type="fixed">
     <parent link="world" />
@@ -64,12 +63,12 @@
       <origin xyz="0 0 0" rpy="0 0 0"/>
       <geometry>
-        <box size="0.01 1.599 1.1" rpy="0 0 0"/>
-      </geometry>
-      <material name="transparent" />
-    </visual>
-    <collision>
-      <origin xyz="0 0 0" rpy="0 0 0"/>
-      <geometry>
-        <box size="0.01 1.599 1.1" rpy="0 0 0"/>
+        <box size="0.01 0.8 0.55" rpy="0 0 0"/>
+      </geometry>
+      <material name="transparent" />
+    </visual>
+    <collision>
+      <origin xyz="0 0 0" rpy="0 0 0"/>
+      <geometry>
+        <box size="0.01 1.6 1.1" rpy="0 0 0"/>
       </geometry>
       <material name="transparent" />
@@ -80,12 +79,12 @@
       <origin xyz="0 0 0" rpy="0 0 0"/>
       <geometry>
-        <box size="0.01 1.599 1.1" rpy="0 0 0"/>
-      </geometry>
-      <material name="transparent" />
-    </visual>
-    <collision>
-      <origin xyz="0 0 0" rpy="0 0 0"/>
-      <geometry>
-        <box size="0.01 1.599 1.1" rpy="0 0 0"/>
+        <box size="0.01 0.8 0.55" rpy="0 0 0"/>
+      </geometry>
+      <material name="transparent" />
+    </visual>
+    <collision>
+      <origin xyz="0 0 0" rpy="0 0 0"/>
+      <geometry>
+        <box size="0.01 1.6 1.1" rpy="0 0 0"/>
       </geometry>
       <material name="transparent" />
@@ -96,12 +95,12 @@
       <origin xyz="0 0 0" rpy="0 0 0"/>
       <geometry>
-        <box size="1.199 0.01 1.1" rpy="0 0 0"/>
-      </geometry>
-      <material name="transparent" />
-    </visual>
-    <collision>
-      <origin xyz="0 0 0" rpy="0 0 0"/>
-      <geometry>
-        <box size="1.199 0.01 1.1" rpy="0 0 0"/>
+        <box size="0.6 0.01 0.55" rpy="0 0 0"/>
+      </geometry>
+      <material name="transparent" />
+    </visual>
+    <collision>
+      <origin xyz="0 0 0" rpy="0 0 0"/>
+      <geometry>
+        <box size="1.2 0.01 1.1" rpy="0 0 0"/>
       </geometry>
       <material name="transparent" />
@@ -112,12 +111,12 @@
       <origin xyz="0 0 0" rpy="0 0 0"/>
       <geometry>
-        <box size="1.199 0.01 1.1" rpy="0 0 0"/>
-      </geometry>
-      <material name="transparent" />
-    </visual>
-    <collision>
-      <origin xyz="0 0 0" rpy="0 0 0"/>
-      <geometry>
-        <box size="1.199 0.01 1.1" rpy="0 0 0"/>
+        <box size="0.6 0.01 0.55" rpy="0 0 0"/>
+      </geometry>
+      <material name="transparent" />
+    </visual>
+    <collision>
+      <origin xyz="0 0 0" rpy="0 0 0"/>
+      <geometry>
+        <box size="1.2 0.01 1.1" rpy="0 0 0"/>
       </geometry>
       <material name="transparent" />
